Commit message: added imu_link

File: src/slam/wheelchair_slam/config/wheelchair_robot.urdf (robot description, URDF)
Before this commit: robot wheelchair_robot, 8 links, 7 joints
Links:
- added link imu_link
Joints:
- added joint base_imu_joint: type fixed, parent imu_link, child base_link, origin xyz=0 0 0 rpy=1.5707963 -1.5707963 0, axis 0 0 1

Commit message: imu offset

File: src/slam/wheelchair_slam/config/wheelchair_robot.urdf (robot description, URDF)
Before this commit: robot wheelchair_robot, 9 links, 8 joints
Joints:
- joint base_imu_joint: origin xyz=0 0 0 rpy=1.5707963 -1.5707963 0 -> xyz=0.09 0 0 rpy=1.5707963 -1.5707963 0

Commit message: made compatible with orbslam

File: src/slam/wheelchair_slam/config/wheelchair_robot.urdf (robot description, URDF)
Before this commit: robot wheelchair_robot, 9 links, 8 joints
Links:
- removed link imu_link
Joints:
- removed joint base_imu_joint
- joint base_camera_joint: origin xyz=0 0 0.32 rpy=0 0 0 -> xyz=0 0 1.3 rpy=0 0 0
